Commit message: Color order is Black-Red-Green-Blue, and overlap visuals

File: vine_robot.urdf (robot description, URDF)
Before this commit: robot vine_robot, 7 links, 6 joints
Joints:
- joint prismatic_joint_0: origin xyz=0.1 0.0 0.0 rpy=0.0 0.0 0.0 -> xyz=0.0 0.0 0.0 rpy=0.0 0.0 0.0
- joint prismatic_joint_1: origin xyz=0.1 0.0 0.0 rpy=0.0 0.0 0.0 -> xyz=0.0 0.0 0.0 rpy=0.0 0.0 0.0
- joint prismatic_joint_2: origin xyz=0.1 0.0 0.0 rpy=0.0 0.0 0.0 -> xyz=0.0 0.0 0.0 rpy=0.0 0.0 0.0

Commit message: Update joint limits

File: vine_robot.urdf (robot description, URDF)
Before this commit: robot vine_robot, 7 links, 6 joints
Joints:
- joint revolute_joint_1: limit lower=-3.146 upper=3.146 effort=10 velocity=3 -> lower=-0.524 upper=0.524 effort=10 velocity=3
- joint revolute_joint_2: limit lower=-3.146 upper=3.146 effort=10 velocity=3 -> lower=-0.524 upper=0.524 effort=10 velocity=3

Commit message: Change links from cubes to cylinders and improve other modeling

File: vine_robot.urdf (robot description, URDF)
Before this commit: robot vine_robot, 7 links, 6 joints
Links:
- link base_link: geometry collision cylinder length=0.1 radius=0.025; visual cylinder length=0.1 radius=0.025
- link link_0: geometry collision cylinder length=0.1 radius=0.025; visual cylinder length=0.1 radius=0.025
- link link_1: geometry collision cylinder length=0.1 radius=0.025; visual cylinder length=0.1 radius=0.025
- link link_2: geometry collision cylinder length=0.1 radius=0.025; visual cylinder length=0.1 radius=0.025
Joints:
- joint prismatic_joint_0: limit lower=0.0 upper=0.5 effort=200 velocity=0.2 -> lower=0.0 upper=1.0 effort=200 velocity=0.1
- joint prismatic_joint_1: limit lower=0.0 upper=0.5 effort=200 velocity=0.2 -> lower=0.0 upper=1.0 effort=200 velocity=0.1
- joint prismatic_joint_2: limit lower=0.0 upper=0.5 effort=200 velocity=0.2 -> lower=0.0 upper=1.0 effort=200 velocity=0.1
- joint revolute_joint_1: limit lower=-0.524 upper=0.524 effort=10 velocity=3 -> lower=-0.5236 upper=0.5236 effort=10 velocity=3
- joint revolute_joint_2: limit lower=-0.524 upper=0.524 effort=10 velocity=3 -> lower=-0.5236 upper=0.5236 effort=10 velocity=3

Commit message: Reduce prismatic joint limit

File: vine_robot.urdf (robot description, URDF)
Before this commit: robot vine_robot, 7 links, 6 joints
Joints:
- joint prismatic_joint_0: limit lower=0.0 upper=1.0 effort=200 velocity=0.1 -> lower=0.0 upper=0.5 effort=200 velocity=0.1
- joint prismatic_joint_1: limit lower=0.0 upper=1.0 effort=200 velocity=0.1 -> lower=0.0 upper=0.5 effort=200 velocity=0.1
- joint prismatic_joint_2: limit lower=0.0 upper=1.0 effort=200 velocity=0.1 -> lower=0.0 upper=0.5 effort=200 velocity=0.1
